Commit message: rune

File: src/rm_gimbal_description/urdf/rm_gimbal.urdf.xacro (robot description, xacro)
@@ -16,5 +16,5 @@
   <link name="camera_link" />
   <joint name="camera_joint" type="fixed">
-    <origin xyz="0.085 0.000 0.035" rpy="0.0  -${pi / 360}  -${0.0}" />
+    <origin xyz="0.085 0.000  0.035" rpy="0.0  ${pi / 360}  ${pi / 120}" />
     <parent link="gimbal_link" />
     <child link="camera_link" />
